Commit message: feat: add initial project files including README, LICENSE, and contribution guidelines

File: urdf/LE1000-URDF-T4.urdf.xacro (robot description, xacro)
@@ -23,9 +23,23 @@
     <visual>
       <origin
-        xyz="0 0 0"
+        xyz="0 0 0.175"
         rpy="0 0 0" />
       <geometry>
         <box
-          size="0.60 0.95 0.70" />
+          size="0.60 0.95 0.35" />
+      </geometry>
+      <material
+        name="">
+        <color
+          rgba="1 1 1 1" />
+      </material>
+    </visual>
+    <visual>
+      <origin
+        xyz="0 0 -0.175"
+        rpy="0 0 0" />
+      <geometry>
+        <box
+          size="0.60 0.90 0.35" />
       </geometry>
       <material
@@ -37,9 +51,18 @@
     <collision>
       <origin
-        xyz="0 0 0"
+        xyz="0 0 0.175"
         rpy="0 0 0" />
       <geometry>
         <box
-          size="0.60 0.95 0.70" />
+          size="0.60 0.95 0.35" />
+      </geometry>
+    </collision>
+    <collision>
+      <origin
+        xyz="0 0 -0.175"
+        rpy="0 0 0" />
+      <geometry>
+        <box
+          size="0.60 0.90 0.35" />
       </geometry>
     </collision>
