Commit message: feat: update URDF configuration with detailed joint definitions and add ros2_control integration

File: urdf/le1000_urdf_t4.urdf.xacro (robot description, xacro)
@@ -3,6 +3,135 @@
      Commit Version: 1.6.0-4-g7f85cfe  Build Version: 1.6.7995.38578
      For more information, please see http://wiki.ros.org/sw_urdf_exporter -->
+<!--
+  Merged with the loone_asv control-layer draft. Real vehicle layout (per team
+  description, corrects earlier guesses in this file's history):
+    * Twin-float catamaran. base_link is the main body/deck, real CAD data
+      from SolidWorks (see urdf/le1000_urdf_t4.csv for the exporter's raw
+      dump), sitting between the two floats.
+    * EACH float has its own propeller and its own rudder (4 actuated joints
+      total, not a single shared unit).
+    * The exported "Joint1"/"Joint2" meshed links ARE the two real rudders
+      (SW component names "Fishtail rudder-1/2" were accurate after all) -
+      one per float. Renamed below to rudder_l_link/rudder_r_link.
+    * float_l_link/float_r_link (pontoon bodies) and propeller_l_link/
+      propeller_r_link have no CAD mesh yet, so they're placeholder
+      primitives, but dimensions/positions below are real team measurements
+      cross-checked against the full boat mesh (base_link.STL, 268 MB -
+      lives outside this repo at the team's CAD export location, too large
+      to check in; NOT shipped as a package asset). That mesh has no
+      separate rudder or camera parts (assembly stand-ins only) but does
+      include the floats and propellers baked into one static shape, which
+      is what the cross-check below is based on:
+        - float_x (0.20955 m) = the real rudder mount X; the mesh confirms
+          each float is centered on that same X.
+        - float_width/length/height (0.125 / 0.834 / 0.259 m) and
+          float_end_height (0.122 m, the tapered section that gives the
+          propeller clearance) are team measurements. float_end_length
+          (0.13 m, the tapered section's own length) is estimated from
+          where the mesh's height taper actually starts/ends.
+        - float_z = 0 (the main float box vertically centered on
+          base_link's own origin) is inferred, not measured directly - but
+          it makes the derived camera-mast top (via head_to_float_top
+          below) land within 2 mm of the mesh's true topmost point (Z =
+          0.477), so it's a well cross-checked placeholder.
+        - propeller Y/Z (0.374 / -0.173 m) come directly from the mesh's
+          propeller-hub region. Independently, the team's "top of rudder to
+          middle of propeller = 0.198 m" measurement matches the straight-
+          line distance between the mesh's rudder-top point and this
+          propeller position to within 2%.
+      TODO(team): replace float/propeller placeholders with real per-part
+      geometry once the rudder/camera/propeller are modeled as separate
+      CAD parts (they're currently only assemblies inside base_link.STL).
+    * Two ZED X cameras sit fixed on top of the main body (base_link), not
+      on the rudder meshes. Body box sized from the ZED X spec sheet
+      (164 x 32 x 37 mm, 120 mm stereo baseline); swap in zedx_mini_size
+      below if a mount actually uses the smaller ZED X variant (94 x 32 x 37
+      mm, 50 mm baseline). The stereo baseline is internal to the camera
+      housing and isn't modeled separately.
+    * The two cameras face opposite directions (e.g. front/rear coverage),
+      cam_span = 0.246 m apart measured face-to-face including the camera
+      bodies themselves (per team measurement) - modeled here as a
+      front/rear pair along Y, each rotated 180 deg in yaw from the other.
+      Vertical placement is derived from a second team measurement: 0.349 m
+      from the top of the camera mast ("top of the head") down to the top
+      of a float - see float_z note above for how well that lines up with
+      the real mesh.
+    * Left/right assignment (J1 => left, J2 => right) is an unverified
+      guess. Swap the _l/_r suffixes below if backwards.
+  ros2_control interface note: propeller_l_joint/propeller_r_joint use the
+  "position" interface even though they're `continuous` - the commanded
+  value is a normalized [0,1] thrust fraction sent to a PCA9685 servo/ESC
+  channel, not a real angle. rudder_l_joint/rudder_r_joint use real radians.
+-->
 <robot
-  name="LE1000-URDF-T4">
+   xmlns:xacro="http://wiki.ros.org/xacro" name="loone_asv">
+  <material name="hull_grey"><color rgba="0.3 0.3 0.35 1.0"/></material>
+  <material name="dark_trim"><color rgba="0.1 0.1 0.1 1.0"/></material>
+  <!-- Float layout: centerline X from the real rudder mount (mesh-confirmed), gap measured by the team. -->
+  <xacro:property name="float_x" value="0.20955"/>
+  <xacro:property name="float_gap" value="0.263"/>
+  <!-- Team measurements (float body + tapered propeller-clearance section). -->
+  <xacro:property name="float_width" value="0.125"/>
+  <xacro:property name="float_length" value="0.834"/>
+  <xacro:property name="float_height" value="0.259"/>
+  <xacro:property name="float_end_height" value="0.122"/>
+  <!-- TODO(team): tapered section's own length is estimated from the mesh, not directly measured. -->
+  <xacro:property name="float_end_length" value="0.13"/>
+  <!-- Inferred (not directly measured) - see top-of-file note for the cross-check. -->
+  <xacro:property name="float_z" value="0"/>
+  <xacro:property name="float_top_z" value="${float_z + float_height / 2}"/>
+  <!-- Main box centered short of the tapered end; both keep the same top (see macro below). -->
+  <xacro:property name="float_main_length" value="${float_length - float_end_length}"/>
+  <xacro:property name="float_main_y" value="${-float_end_length / 2}"/>
+  <xacro:property name="float_end_y" value="${float_length / 2 - float_end_length / 2}"/>
+  <!-- Propeller hub position, from the base_link.STL mesh (see top-of-file note). -->
+  <xacro:property name="prop_y" value="0.374"/>
+  <xacro:property name="prop_z" value="-0.173"/>
+  <!-- Central body box width, from the mesh: the original 0.60 m box spanned the whole
+       boat (both floats included), which now double-draws against float_l/r_link above.
+       0.22 m is where the mesh's dense central hull cluster actually ends (x ~ +/-0.11). -->
+  <xacro:property name="hull_width" value="0.22"/>
+  <!-- ZED X body box, from the spec sheet (length x depth x height). -->
+  <xacro:property name="zedx_length" value="0.164"/>
+  <xacro:property name="zedx_depth" value="0.032"/>
+  <xacro:property name="zedx_height" value="0.037"/>
+  <xacro:property name="zedx_size" value="${zedx_length} ${zedx_depth} ${zedx_height}"/>
+  <xacro:property name="zedx_mini_size" value="0.094 0.032 0.037"/>
+  <!-- Cameras face opposite directions along Y; span is face-to-face including
+       the camera bodies (team measurement), so each box center sits half a
+       camera-depth in from the outer face. -->
+  <xacro:property name="cam_span" value="0.246"/>
+  <xacro:property name="cam_y" value="${(cam_span - zedx_depth) / 2}"/>
+  <!-- Vertical placement chains off float_top_z above (team measurement). -->
+  <xacro:property name="head_to_float_top" value="0.349"/>
+  <xacro:property name="cam_top_z" value="${float_top_z + head_to_float_top}"/>
+  <xacro:property name="cam_z" value="${cam_top_z - zedx_height / 2}"/>
+  <xacro:macro name="zedx_body">
+    <visual>
+      <origin xyz="0 0 0" rpy="0 0 0" />
+      <geometry>
+        <box size="${zedx_size}" />
+      </geometry>
+      <material name="dark_trim"/>
+    </visual>
+  </xacro:macro>
+  <!-- Float body: main box plus a shorter/thinner box at the propeller end,
+       both top-aligned so the underside steps up for propeller clearance. -->
+  <xacro:macro name="float_body">
+    <visual>
+      <origin xyz="0 ${float_main_y} 0" rpy="0 0 0"/>
+      <geometry>
+        <box size="${float_width} ${float_main_length} ${float_height}"/>
+      </geometry>
+      <material name="hull_grey"/>
+    </visual>
+    <visual>
+      <origin xyz="0 ${float_end_y} ${(float_height - float_end_height) / 2}" rpy="0 0 0"/>
+      <geometry>
+        <box size="${float_width} ${float_end_length} ${float_end_height}"/>
+      </geometry>
+      <material name="hull_grey"/>
+    </visual>
+  </xacro:macro>
   <link
     name="base_link">
@@ -27,11 +156,8 @@
       <geometry>
         <box
-          size="0.60 0.95 0.35" />
+          size="${hull_width} 0.95 0.35" />
       </geometry>
       <material
-        name="">
-        <color
-          rgba="1 1 1 1" />
-      </material>
+        name="hull_grey"/>
     </visual>
     <visual>
@@ -41,11 +167,8 @@
       <geometry>
         <box
-          size="0.60 0.90 0.35" />
+          size="${hull_width} 0.90 0.35" />
       </geometry>
       <material
-        name="">
-        <color
-          rgba="1 1 1 1" />
-      </material>
+        name="hull_grey"/>
     </visual>
     <collision>
@@ -55,5 +178,5 @@
       <geometry>
         <box
-          size="0.60 0.95 0.35" />
+          size="${hull_width} 0.95 0.35" />
       </geometry>
     </collision>
@@ -64,10 +187,24 @@
       <geometry>
         <box
-          size="0.60 0.90 0.35" />
+          size="${hull_width} 0.90 0.35" />
       </geometry>
     </collision>
   </link>
+  <!-- ============================ Floats (placeholder shape, real measured dimensions) ============================ -->
+  <link name="float_l_link"><xacro:float_body/></link>
+  <link name="float_r_link"><xacro:float_body/></link>
+  <joint name="float_l_joint" type="fixed">
+    <parent link="base_link"/>
+    <child link="float_l_link"/>
+    <origin xyz="${float_x} 0 ${float_z}" rpy="0 0 0"/>
+  </joint>
+  <joint name="float_r_joint" type="fixed">
+    <parent link="base_link"/>
+    <child link="float_r_link"/>
+    <origin xyz="${-float_x} 0 ${float_z}" rpy="0 0 0"/>
+  </joint>
+  <!-- ============================ Rudders (real CAD, one per float) ============================ -->
   <link
-    name="Joint1">
+    name="rudder_l_link">
     <inertial>
       <origin
@@ -93,8 +230,5 @@
       </geometry>
       <material
-        name="">
-        <color
-          rgba="1 1 1 1" />
-      </material>
+        name="dark_trim"/>
     </visual>
     <collision>
@@ -109,5 +243,5 @@
   </link>
   <joint
-    name="J1"
+    name="rudder_l_joint"
     type="revolute">
     <origin
@@ -117,15 +251,16 @@
       link="base_link" />
     <child
-      link="Joint1" />
+      link="rudder_l_link" />
     <axis
       xyz="0 -1 0" />
+    <!-- TODO(team): placeholder range; confirm against the real servo/linkage throw. -->
     <limit
-      lower="0"
-      upper="0"
-      effort="0"
-      velocity="0" />
+      lower="-0.6"
+      upper="0.6"
+      effort="5.0"
+      velocity="3.0" />
   </joint>
   <link
-    name="Joint2">
+    name="rudder_r_link">
     <inertial>
       <origin
@@ -151,8 +286,5 @@
       </geometry>
       <material
-        name="">
-        <color
-          rgba="1 1 1 1" />
-      </material>
+        name="dark_trim"/>
     </visual>
     <collision>
@@ -167,5 +299,5 @@
   </link>
   <joint
-    name="J2"
+    name="rudder_r_joint"
     type="revolute">
     <origin
@@ -175,12 +307,76 @@
       link="base_link" />
     <child
-      link="Joint2" />
+      link="rudder_r_link" />
     <axis
       xyz="0 -1 0" />
     <limit
-      lower="0"
-      upper="0"
-      effort="0"
-      velocity="0" />
-  </joint>
+      lower="-0.6"
+      upper="0.6"
+      effort="5.0"
+      velocity="3.0" />
+  </joint>
+  <!-- ============================ Propellers (placeholder shape, mesh-derived position) ============================ -->
+  <!-- Modeled as `continuous` so ros2_control can expose a command interface; the
+       numeric command is a normalized [0,1] thrust fraction, NOT a real angle. -->
+  <link name="propeller_l_link"><visual><geometry><cylinder radius="0.05" length="0.08"/></geometry><material name="dark_trim"/></visual></link>
+  <link name="propeller_r_link"><visual><geometry><cylinder radius="0.05" length="0.08"/></geometry><material name="dark_trim"/></visual></link>
+  <joint name="propeller_l_joint" type="continuous">
+    <parent link="base_link"/>
+    <child link="propeller_l_link"/>
+    <origin xyz="${float_x} ${prop_y} ${prop_z}" rpy="0 1.5708 0"/>
+    <axis xyz="0 0 1"/>
+  </joint>
+  <joint name="propeller_r_joint" type="continuous">
+    <parent link="base_link"/>
+    <child link="propeller_r_link"/>
+    <origin xyz="${-float_x} ${prop_y} ${prop_z}" rpy="0 1.5708 0"/>
+    <axis xyz="0 0 1"/>
+  </joint>
+  <!-- ============================ Cameras (placeholder, on top of main body) ============================ -->
+  <link name="cam_1_link">
+    <xacro:zedx_body/>
+  </link>
+  <link name="cam_2_link">
+    <xacro:zedx_body/>
+  </link>
+  <joint name="cam_1_joint" type="fixed">
+    <parent link="base_link"/>
+    <child link="cam_1_link"/>
+    <origin xyz="0 ${cam_y} ${cam_z}" rpy="0 0 0"/>
+  </joint>
+  <joint name="cam_2_joint" type="fixed">
+    <parent link="base_link"/>
+    <child link="cam_2_link"/>
+    <origin xyz="0 ${-cam_y} ${cam_z}" rpy="0 0 3.14159"/>
+  </joint>
+  <!-- ============================ ros2_control ============================ -->
+  <!--
+    Stock topic_based_ros2_control hardware: it bridges the command/state interfaces
+    below to plain ROS topics instead of a real driver, so the actual PCA9685 access
+    can live in a Python driver node (no C++) subscribed to joint_commands_topic and
+    publishing joint_states_topic.
+  -->
+  <ros2_control name="asv" type="system">
+    <hardware>
+      <plugin>topic_based_ros2_control/TopicBasedSystem</plugin>
+      <param name="joint_commands_topic">/asv/joint_commands</param>
+      <param name="joint_states_topic">/asv/joint_states</param>
+    </hardware>
+    <joint name="propeller_l_joint">
+      <command_interface name="position"/>
+      <state_interface name="position"/>
+    </joint>
+    <joint name="propeller_r_joint">
+      <command_interface name="position"/>
+      <state_interface name="position"/>
+    </joint>
+    <joint name="rudder_l_joint">
+      <command_interface name="position"/>
+      <state_interface name="position"/>
+    </joint>
+    <joint name="rudder_r_joint">
+      <command_interface name="position"/>
+      <state_interface name="position"/>
+    </joint>
+  </ros2_control>
 </robot>

Commit message: feat: refine URDF propeller and camera mast definitions for accurate positioning

File: urdf/le1000_urdf_t4.urdf.xacro (robot description, xacro)
@@ -35,12 +35,24 @@
           below) land within 2 mm of the mesh's true topmost point (Z =
           0.477), so it's a well cross-checked placeholder.
-        - propeller Y/Z (0.374 / -0.173 m) come directly from the mesh's
+        - propeller Y (0.374 m) and the raw propeller Z reading (-0.173 m,
+          kept as prop_z_measured) come directly from the mesh's
           propeller-hub region. Independently, the team's "top of rudder to
           middle of propeller = 0.198 m" measurement matches the straight-
           line distance between the mesh's rudder-top point and this
           propeller position to within 2%.
+        - prop_z itself is then moved up from that raw reading to sit flush
+          against the float's tapered underside (float_tapered_bottom_z
+          minus the propeller radius) instead of hanging below it with a
+          visible gap. rudder_mount_z gets the exact same upward shift
+          (rudder_z_shift) applied to its real CAD Z (rudder_mount_z_measured),
+          so the measured 0.198 m rudder-to-propeller relationship is
+          preserved even though both moved.
       TODO(team): replace float/propeller placeholders with real per-part
       geometry once the rudder/camera/propeller are modeled as separate
       CAD parts (they're currently only assemblies inside base_link.STL).
+    * cam_mast_link is a thin placeholder box connecting the hull top
+      (hull_top_z) to the cameras (cam_bottom_z) - without it the cameras
+      rendered floating in mid-air above the hull with nothing visibly
+      holding them up.
     * Two ZED X cameras sit fixed on top of the main body (base_link), not
       on the rudder meshes. Body box sized from the ZED X spec sheet
@@ -85,11 +97,30 @@
   <xacro:property name="float_main_y" value="${-float_end_length / 2}"/>
   <xacro:property name="float_end_y" value="${float_length / 2 - float_end_length / 2}"/>
-  <!-- Propeller hub position, from the base_link.STL mesh (see top-of-file note). -->
+  <!-- Propeller hub position: Y is from the base_link.STL mesh (see top-of-file note).
+       Z is tucked flush against the float's tapered underside instead of the raw mesh
+       reading (prop_z_measured), which left a visible gap between propeller and float.
+       The same delta is then applied to the rudder mount below so the real measured
+       0.198 m top-of-rudder-to-propeller relationship is preserved, not just the
+       propeller moved in isolation. -->
+  <xacro:property name="propeller_radius" value="0.05"/>
   <xacro:property name="prop_y" value="0.374"/>
-  <xacro:property name="prop_z" value="-0.173"/>
-  <!-- Central body box width, from the mesh: the original 0.60 m box spanned the whole
-       boat (both floats included), which now double-draws against float_l/r_link above.
-       0.22 m is where the mesh's dense central hull cluster actually ends (x ~ +/-0.11). -->
+  <xacro:property name="prop_z_measured" value="-0.173"/>
+  <xacro:property name="float_tapered_bottom_z" value="${float_top_z - float_end_height}"/>
+  <xacro:property name="prop_z" value="${float_tapered_bottom_z - propeller_radius}"/>
+  <xacro:property name="rudder_z_shift" value="${prop_z - prop_z_measured}"/>
+  <!-- Real CAD mount Z from the SolidWorks export, plus the same shift as the propeller above. -->
+  <xacro:property name="rudder_mount_z_measured" value="-0.06586"/>
+  <xacro:property name="rudder_mount_z" value="${rudder_mount_z_measured + rudder_z_shift}"/>
+  <!-- Central body box, from the mesh (base_link.STL, |x| <= 0.11 slice): the original
+       two stacked boxes (0.60 m wide, z spanning -0.35 to +0.35, y spanning ~0.9-0.95)
+       were sized to the WHOLE boat's outer envelope (floats included), not just the
+       central body between them. That's now redundant with float_l/r_link above and,
+       worse, left a box hanging in mid-air below the real hull (the actual center only
+       dips to z ~ -0.07). Replaced with a single box sized to the central body alone;
+       still a placeholder shape, but the real cross-checked extent, not a guess. -->
   <xacro:property name="hull_width" value="0.22"/>
+  <xacro:property name="hull_length" value="0.60"/>
+  <xacro:property name="hull_height" value="0.37"/>
+  <xacro:property name="hull_z" value="0.115"/>
   <!-- ZED X body box, from the spec sheet (length x depth x height). -->
   <xacro:property name="zedx_length" value="0.164"/>
@@ -107,4 +138,13 @@
   <xacro:property name="cam_top_z" value="${float_top_z + head_to_float_top}"/>
   <xacro:property name="cam_z" value="${cam_top_z - zedx_height / 2}"/>
+  <!-- Mast connecting the hull top to the cameras (otherwise they render floating in
+       mid-air, since cam_z sits well above hull_top_z). Placeholder box, thin in X,
+       wide enough in Y to sit under both front/rear-facing camera footprints. -->
+  <xacro:property name="hull_top_z" value="${hull_z + hull_height / 2}"/>
+  <xacro:property name="cam_bottom_z" value="${cam_z - zedx_height / 2}"/>
+  <xacro:property name="mast_width" value="${hull_width}"/>
+  <xacro:property name="mast_length" value="${2 * cam_y + zedx_depth}"/>
+  <xacro:property name="mast_height" value="${cam_bottom_z - hull_top_z}"/>
+  <xacro:property name="mast_z" value="${(hull_top_z + cam_bottom_z) / 2}"/>
   <xacro:macro name="zedx_body">
     <visual>
@@ -152,40 +192,20 @@
     <visual>
       <origin
-        xyz="0 0 0.175"
+        xyz="0 0 ${hull_z}"
         rpy="0 0 0" />
       <geometry>
         <box
-          size="${hull_width} 0.95 0.35" />
+          size="${hull_width} ${hull_length} ${hull_height}" />
       </geometry>
       <material
         name="hull_grey"/>
     </visual>
-    <visual>
-      <origin
-        xyz="0 0 -0.175"
+    <collision>
+      <origin
+        xyz="0 0 ${hull_z}"
         rpy="0 0 0" />
       <geometry>
         <box
-          size="${hull_width} 0.90 0.35" />
-      </geometry>
-      <material
-        name="hull_grey"/>
-    </visual>
-    <collision>
-      <origin
-        xyz="0 0 0.175"
-        rpy="0 0 0" />
-      <geometry>
-        <box
-          size="${hull_width} 0.95 0.35" />
-      </geometry>
-    </collision>
-    <collision>
-      <origin
-        xyz="0 0 -0.175"
-        rpy="0 0 0" />
-      <geometry>
-        <box
-          size="${hull_width} 0.90 0.35" />
+          size="${hull_width} ${hull_length} ${hull_height}" />
       </geometry>
     </collision>
@@ -246,5 +266,5 @@
     type="revolute">
     <origin
-      xyz="0.20955 0.47374 -0.06586"
+      xyz="0.20955 0.47374 ${rudder_mount_z}"
       rpy="1.5708 0 1.5708" />
     <parent
@@ -302,5 +322,5 @@
     type="revolute">
     <origin
-      xyz="-0.20955 0.47374 -0.06586"
+      xyz="-0.20955 0.47374 ${rudder_mount_z}"
       rpy="1.5708 0 1.5708" />
     <parent
@@ -319,6 +339,6 @@
   <!-- Modeled as `continuous` so ros2_control can expose a command interface; the
        numeric command is a normalized [0,1] thrust fraction, NOT a real angle. -->
-  <link name="propeller_l_link"><visual><geometry><cylinder radius="0.05" length="0.08"/></geometry><material name="dark_trim"/></visual></link>
-  <link name="propeller_r_link"><visual><geometry><cylinder radius="0.05" length="0.08"/></geometry><material name="dark_trim"/></visual></link>
+  <link name="propeller_l_link"><visual><geometry><cylinder radius="${propeller_radius}" length="0.08"/></geometry><material name="dark_trim"/></visual></link>
+  <link name="propeller_r_link"><visual><geometry><cylinder radius="${propeller_radius}" length="0.08"/></geometry><material name="dark_trim"/></visual></link>
   <joint name="propeller_l_joint" type="continuous">
     <parent link="base_link"/>
@@ -333,5 +353,11 @@
     <axis xyz="0 0 1"/>
   </joint>
-  <!-- ============================ Cameras (placeholder, on top of main body) ============================ -->
+  <!-- ============================ Camera mast + cameras (placeholder, on top of main body) ============================ -->
+  <link name="cam_mast_link"><visual><geometry><box size="${mast_width} ${mast_length} ${mast_height}"/></geometry><material name="hull_grey"/></visual></link>
+  <joint name="cam_mast_joint" type="fixed">
+    <parent link="base_link"/>
+    <child link="cam_mast_link"/>
+    <origin xyz="0 0 ${mast_z}" rpy="0 0 0"/>
+  </joint>
   <link name="cam_1_link">
     <xacro:zedx_body/>
