Commit message: feat: add complete URDF description for Loon-E ASV with detailed links and joints

File: urdf/loone_asv.export.urdf (robot description, URDF)
Before this commit: robot loone_asv, 4 links, 3 joints
Links:
- link base_link: geometry collision box size=1.0 0.6 0.2; visual box size=1.0 0.6 0.2
Joints:
- joint prop_l_joint: origin xyz=${prop_x} ${prop_y} 0 rpy=0 1.5708 0 -> xyz=-0.45 0.25 0 rpy=0 1.5708 0
- joint prop_r_joint: origin xyz=${prop_x} ${-prop_y} 0 rpy=0 1.5708 0 -> xyz=-0.45 -0.25 0 rpy=0 1.5708 0
- joint rudder_joint: axis 0 0 1 -> 0 0 0; origin xyz=${rudder_x} 0 0 rpy=0 0 1.5708 -> xyz=-0.55 0 0 rpy=0 0 1.5708
