Commit message: feat: add GPS link and joint for accurate positioning

File: urdf/loone_asv.urdf.xacro (robot description, xacro)
@@ -55,4 +55,9 @@
   <link name="prop_r_link"><visual><geometry><cylinder radius="0.05" length="0.08"/></geometry><material name="prop_dark"/></visual></link>
   <link name="rudder_link"><visual><geometry><box size="0.02 0.05 0.15"/></geometry><material name="prop_dark"/></visual></link>
+  <!-- GPS antenna mount, frame-only (no geometry). TODO(team): measure the real
+       offset if the antenna ever isn't at the boat's origin. phone.py stamps its
+       NavSatFix messages with this frame, and navsat_transform_node uses the offset
+       between it and base_link to place the GPS fix correctly. -->
+  <link name="gps_link"/>
   <!-- ============================ Joints ============================ -->
   <!-- The propellers spin about their thrust axis. We model them as `continuous`
@@ -79,4 +84,9 @@
     <axis xyz="0 0 1"/>
     <limit lower="-0.6" upper="0.6" effort="5.0" velocity="3.0"/>
+  </joint>
+  <joint name="gps_joint" type="fixed">
+    <parent link="base_link"/>
+    <child link="gps_link"/>
+    <origin xyz="0 0 0" rpy="0 0 0"/>
   </joint>
   <!-- ============================ ros2_control ============================ -->

Commit message: feat: refine URDF for Loon-E ASV with updated properties, links, and joints

File: urdf/loone_asv.urdf.xacro (robot description, xacro)
@@ -30,11 +30,13 @@
   <xacro:property name="hull_width"  value="0.6"/>   <!-- m -->
   <xacro:property name="hull_height" value="0.2"/>   <!-- m -->
-  <xacro:property name="prop_x"      value="-0.45"/> <!-- props near the stern -->
-  <xacro:property name="prop_y"      value="0.25"/>  <!-- half the thruster separation -->
-  <xacro:property name="rudder_x"    value="-0.55"/> <!-- rudder behind the props -->
+  <xacro:property name="prop_x"      value="-0.40"/> <!-- props near the stern -->
+  <xacro:property name="prop_y"      value="0.209"/>  <!-- half the thruster separation -->
+  <xacro:property name="prop_z"      value="-0.169"/>   <!-- props at waterline -->
+  <xacro:property name="rudder_x"    value="-0.47"/> <!-- rudder behind the props -->
+  <xacro:property name="rudder_z"    value="-0.065"/>   <!-- rudder height -->
+  <!-- ============================ Materials ============================ -->
   <material name="hull_grey"><color rgba="0.3 0.3 0.35 1.0"/></material>
   <material name="prop_dark"><color rgba="0.1 0.1 0.1 1.0"/></material>
   <!-- ============================ Links ============================ -->
-  <!-- base_link: the robot base frame nav2 plans for. Origin ~ boat center. -->
   <link name="base_link">
     <visual>
@@ -57,13 +59,57 @@
     </inertial>
   </link>
-  <!-- Simple placeholder links for the two thrusters and the rudder. -->
-  <link name="prop_l_link"><visual><geometry><cylinder radius="0.05" length="0.08"/></geometry><material name="prop_dark"/></visual></link>
-  <link name="prop_r_link"><visual><geometry><cylinder radius="0.05" length="0.08"/></geometry><material name="prop_dark"/></visual></link>
-  <link name="rudder_link"><visual><geometry><box size="0.02 0.05 0.15"/></geometry><material name="prop_dark"/></visual></link>
+  <link name="prop_l_link">
+    <visual>
+    <origin xyz="0 0 0" rpy="1.5708 0 1.5708"/>
+    <geometry>
+      <cylinder radius="0.05" length="0.08"/>
+    </geometry>
+    <material name="prop_dark"/>
+    </visual>
+  </link>
+  <link name="prop_r_link">
+    <visual>
+      <origin xyz="0 0 0" rpy="1.5708 0 1.5708"/>
+      <geometry>
+        <cylinder radius="0.05" length="0.08"/>
+      </geometry>
+      <material name="prop_dark"/>
+    </visual>
+  </link>
+   <link name="rudder_r_link">
+    <visual>
+     <origin
+        xyz="0 0 0"
+        rpy="1.5708 0 1.5708"/>
+      <geometry>
+        <mesh
+            filename="package://le1000_urdf_t4/meshes/Joint1.STL" />
+      </geometry>
+      <material name="prop_dark"/>
+    </visual>
+  </link>
+  <link name="rudder_l_link">
+    <visual>
+     <origin
+        xyz="0 0 0"
+        rpy="1.5708 0 1.5708"/>
+      <geometry>
+        <mesh
+            filename="package://le1000_urdf_t4/meshes/Joint1.STL" />
+      </geometry>
+      <material name="prop_dark"/>
+    </visual>
+  </link>
   <!-- GPS antenna mount, frame-only (no geometry). TODO(team): measure the real
        offset if the antenna ever isn't at the boat's origin. phone.py stamps its
        NavSatFix messages with this frame, and navsat_transform_node uses the offset
        between it and base_link to place the GPS fix correctly. -->
-  <link name="gps_link"/>
+  <link name="gps_link">
+    <visual>
+      <origin xyz="0 0 0" rpy="0 0 0"/>
+      <geometry><box size="0.01 0.01 0.01"/></geometry>
+      <material name="prop_dark"/>
+    </visual>
+  </link>
   <!-- ============================ Joints ============================ -->
   <!-- The propellers spin about their thrust axis. We model them as `continuous`
@@ -73,5 +119,5 @@
     <parent link="base_link"/>
     <child link="prop_l_link"/>
-    <origin xyz="${prop_x} ${prop_y} 0" rpy="1.5708 0 0"/>
+    <origin xyz="${prop_x} ${prop_y} ${prop_z}" rpy="0 0 3.14159"/>
     <axis xyz="1 0 0"/>
   </joint>
@@ -79,13 +125,20 @@
     <parent link="base_link"/>
     <child link="prop_r_link"/>
-    <origin xyz="${prop_x} ${-prop_y} 0" rpy="1.5708 0 0"/>
+    <origin xyz="${prop_x} ${-prop_y} ${prop_z}" rpy="0 0 3.14159"/>
     <axis xyz="1 0 0"/>
   </joint>
   <!-- Rudder deflects left/right about the vertical axis. `revolute` with generous
        limits; the numeric command is a normalized [0,1] fraction (0.55 ~ straight). -->
-  <joint name="rudder_joint" type="revolute">
+  <joint name="rudder_r_joint" type="revolute">
     <parent link="base_link"/>
-    <child link="rudder_link"/>
-    <origin xyz="${rudder_x} 0 0" rpy="0 0 1.5708"/>
+    <child link="rudder_r_link"/>
+    <origin xyz="${rudder_x} ${-prop_y} ${rudder_z}" rpy="0 0 1.5708"/>
+    <axis xyz="0 0 1"/>
+    <limit lower="-0.6" upper="0.6" effort="5.0" velocity="3.0"/>
+  </joint>
+  <joint name="rudder_l_joint" type="revolute">
+    <parent link="base_link"/>
+    <child link="rudder_l_link"/>
+    <origin xyz="${rudder_x} ${prop_y} ${rudder_z}" rpy="0 0 1.5708"/>
     <axis xyz="0 0 1"/>
     <limit lower="-0.6" upper="0.6" effort="5.0" velocity="3.0"/>
@@ -94,5 +147,5 @@
     <parent link="base_link"/>
     <child link="gps_link"/>
-    <origin xyz="0 0 0" rpy="0 0 0"/>
+    <origin xyz="0 0 0.33" rpy="0 0 0"/>
   </joint>
   <!-- ============================ ros2_control ============================ -->
@@ -127,5 +180,9 @@
       <state_interface name="position"/>
     </joint>
-    <joint name="rudder_joint">
+    <joint name="rudder_r_joint">
+      <command_interface name="position"/>
+      <state_interface name="position"/>
+    </joint>
+    <joint name="rudder_l_joint">
       <command_interface name="position"/>
       <state_interface name="position"/>

Commit message: fix: URDF is now more accure

File: urdf/loone_asv.urdf.xacro (robot description, xacro)
@@ -25,17 +25,40 @@
 <robot xmlns:xacro="http://wiki.ros.org/xacro" name="loone_asv">
   <!-- ============================ Tunable geometry ============================ -->
-  <!-- TODO(team): measure the real boat. These are placeholders just so RViz shows
-       roughly the right shape; only the joint axes matter for control. -->
+  <!-- ============================ Hull geometry ============================ -->
   <xacro:property name="hull_length" value="1.0"/>   <!-- m -->
   <xacro:property name="hull_width"  value="0.6"/>   <!-- m -->
   <xacro:property name="hull_height" value="0.2"/>   <!-- m -->
+  <!-- ============================ Propellers ============================ -->
   <xacro:property name="prop_x"      value="-0.40"/> <!-- props near the stern -->
   <xacro:property name="prop_y"      value="0.209"/>  <!-- half the thruster separation -->
   <xacro:property name="prop_z"      value="-0.169"/>   <!-- props at waterline -->
+  <!-- ============================ Rudder ============================ -->
   <xacro:property name="rudder_x"    value="-0.47"/> <!-- rudder behind the props -->
   <xacro:property name="rudder_z"    value="-0.065"/>   <!-- rudder height -->
+  <!-- ============================ ZEDX ============================ -->
+  <xacro:property name="zedx_length" value="0.164"/>
+  <xacro:property name="zedx_depth" value="0.032"/>
+  <xacro:property name="zedx_height" value="0.037"/>
+  <xacro:property name="zedx_size" value="${zedx_depth} ${zedx_length} ${zedx_height}"/>
+  <xacro:property name="zedx_mini_size" value="0.094 0.032 0.037"/>
+  <!-- ============================ Cameras ============================ -->
+  <xacro:property name="cam_span" value="0.107"/>
+  <xacro:property name="cam_y" value="${0}"/>
+  <xacro:property name="cam_x" value="${cam_span}" />
+  <xacro:property name="cam_top_z" value="${0.350}"/>
+  <xacro:property name="cam_z" value="${cam_top_z - zedx_height / 2}"/>
   <!-- ============================ Materials ============================ -->
   <material name="hull_grey"><color rgba="0.3 0.3 0.35 1.0"/></material>
   <material name="prop_dark"><color rgba="0.1 0.1 0.1 1.0"/></material>
+  <!-- ============================ ZEDx Body ==========================-->
+  <xacro:macro name="zedx_body">
+    <visual>
+      <origin xyz="0 0 0" rpy="0 0 0" />
+      <geometry>
+        <box size="${zedx_size}" />
+      </geometry>
+      <material name="prop_dark"/>
+    </visual>
+  </xacro:macro>
   <!-- ============================ Links ============================ -->
   <link name="base_link">
@@ -112,4 +135,10 @@
     </visual>
   </link>
+  <link name="cam_1_link">
+    <xacro:zedx_body/>
+  </link>
+  <link name="cam_2_link">
+    <xacro:zedx_body/>
+  </link>
   <!-- ============================ Joints ============================ -->
   <!-- The propellers spin about their thrust axis. We model them as `continuous`
@@ -119,5 +148,5 @@
     <parent link="base_link"/>
     <child link="prop_l_link"/>
-    <origin xyz="${prop_x} ${prop_y} ${prop_z}" rpy="0 0 3.14159"/>
+    <origin xyz="${prop_x} ${prop_y} ${prop_z}" rpy="0 0 0"/>
     <axis xyz="1 0 0"/>
   </joint>
@@ -125,5 +154,5 @@
     <parent link="base_link"/>
     <child link="prop_r_link"/>
-    <origin xyz="${prop_x} ${-prop_y} ${prop_z}" rpy="0 0 3.14159"/>
+    <origin xyz="${prop_x} ${-prop_y} ${prop_z}" rpy="0 0 0"/>
     <axis xyz="1 0 0"/>
   </joint>
@@ -148,4 +177,16 @@
     <child link="gps_link"/>
     <origin xyz="0 0 0.33" rpy="0 0 0"/>
+  </joint>
+  <joint name="cam_1_joint" type="fixed">
+    <parent link="base_link"/>
+    <child link="cam_1_link"/>
+    <!-- Stern side (same side as props/rudder): boresight faces +Y (aft). -->
+    <origin xyz="${cam_x} ${cam_y} ${cam_z}" rpy="0 0 0"/>
+  </joint>
+  <joint name="cam_2_joint" type="fixed">
+    <parent link="base_link"/>
+    <child link="cam_2_link"/>
+    <!-- Bow side, confirmed physical front camera: boresight faces -Y (forward). -->
+    <origin xyz="${-cam_x} ${cam_y} ${cam_z}" rpy="0 0 -3.14"/>
   </joint>
   <!-- ============================ ros2_control ============================ -->

Commit message: fix; adjust URDF for zed

File: urdf/loone_asv.urdf.xacro (robot description, xacro)
@@ -6,22 +6,38 @@
     * Declare the three actuated joints (2 propellers + 1 rudder) and expose them
       to ros2_control through the stock topic_based_ros2_control hardware.
-  What this is NOT:
-    * It does not include the ZED camera description. The ZED wrapper already runs
-      its own robot_state_publisher and publishes `odom -> zedx_camera_link`. We
-      connect the camera frame to `base_link` with a single static_transform_publisher
-      in bringup.launch.py instead, so no frame is broadcast by two publishers.
+  THE CAMERA IS THE ROOT OF THIS TREE, AND cam_1 IS THE ZED X
+    This file INCLUDES the ZED wrapper's own zed_macro.urdf.xacro and instantiates
+    it as the root link, so `<camera_name>_camera_link` and its child frames come
+    from Stereolabs' description rather than being approximated here. cam_1 is not
+    a separate placeholder link any more; it IS the ZED X, and its mount offset
+    lives in exactly one place: cam_1_to_base_link below.
+    Because of that, bringup.launch.py passes `publish_urdf:=false` to the wrapper.
+    Left at its default the wrapper starts a SECOND robot_state_publisher
+    (/<ns>/<camera_name>_state_publisher) describing the same camera, which is
+    what previously put two competing robot descriptions on the graph.
+  WHY THE TREE IS INVERTED
+    This wrapper version has no `base_frame` parameter (grep the submodule, there
+    is none), so it can only publish `odom -> <camera_name>_camera_link`. It cannot
+    be told to track base_link. A URDF has exactly one root, and TF allows exactly
+    one parent per frame, so base_link necessarily hangs BELOW the camera. That is
+    unconventional (usually odom -> base_link -> sensors) but TF-valid.
+    The payoff is that no static_transform_publisher is needed at all: the joint
+    below encodes the camera->base_link offset, so the mount geometry cannot drift
+    out of sync with a separate hand-maintained transform the way it used to.
   TF layout produced with the launch file:
       map (SLAM Toolbox)
-        -> odom (ZED)
-          -> zedx_camera_link (ZED)
-            -> base_link            (static_transform_publisher, in bringup.launch.py)
-              -> prop_l / prop_r / rudder links   (this file, via robot_state_publisher)
-  NOTE on the tree shape: ZED publishes odom -> zedx_camera_link directly and this
-  wrapper version has no "base_frame" parameter, so base_link necessarily hangs
-  BELOW the camera. That is unconventional (usually odom -> base_link -> sensors)
-  but TF-valid. If you later want the classic layout, make the ZED track base_link
-  and flip the static transform. See bringup.launch.py TODO.
+        -> odom (ZED wrapper, pos_tracking)
+          -> <camera_name>_camera_link       (ZED macro, THIS file, = cam_1)
+            -> <camera_name>_camera_center -> left/right frames + optical frames
+            -> base_link                    (cam_1_to_base_link, THIS file)
+              -> prop_l / prop_r / rudder_r / rudder_l / gps_link / cam_2_link
 -->
 <robot xmlns:xacro="http://wiki.ros.org/xacro" name="loone_asv">
+  <!-- Must match the camera_name/camera_model passed to the ZED wrapper, or the
+       frames this file declares will not be the ones the wrapper publishes into.
+       bringup.launch.py forwards its own launch arguments here. -->
+  <xacro:arg name="camera_name"  default="zedx"/>
+  <xacro:arg name="camera_model" default="zedx"/>
+  <xacro:include filename="$(find zed_wrapper)/urdf/zed_macro.urdf.xacro"/>
   <!-- ============================ Tunable geometry ============================ -->
   <!-- ============================ Hull geometry ============================ -->
@@ -61,4 +77,25 @@
     </visual>
   </xacro:macro>
+  <!-- ================= ROOT: the ZED X (a.k.a. cam_1) ================= -->
+  <!-- Stereolabs' own macro, so the camera body, baseline and optical frames match
+       what zed_wrapper publishes into. It declares `<name>_camera_link` with no
+       parent, which makes it this robot's root; see the header for why.
+       The <origin> is the macro's required `*gnss_origin` block parameter: xacro
+       demands the block even when enable_gnss is false, in which case it is unused.
+       We keep GNSS off here and use our own gps_link below, because that is the
+       frame phone.py and sim_gnss.py stamp their NavSatFix with. -->
+  <xacro:zed_camera name="$(arg camera_name)" model="$(arg camera_model)">
+    <origin xyz="0 0 0" rpy="0 0 0"/>
+  </xacro:zed_camera>
+  <!-- Camera -> base_link: the INVERSE of where cam_1 sits on the boat.
+       cam_1's mount is (cam_x, cam_y, cam_z) from base_link with no rotation, so
+       the inverse is simply the negated translation. If you ever give this joint a
+       non-zero rpy, the inverse is NO LONGER just negated xyz: you would have to
+       invert the rotation and rotate the translation by it. -->
+  <joint name="cam_1_to_base_link" type="fixed">
+    <parent link="$(arg camera_name)_camera_link"/>
+    <child link="base_link"/>
+    <origin xyz="${-cam_x} ${-cam_y} ${-cam_z}" rpy="0 0 0"/>
+  </joint>
   <!-- ============================ Links ============================ -->
   <link name="base_link">
@@ -135,7 +172,10 @@
     </visual>
   </link>
-  <link name="cam_1_link">
-    <xacro:zedx_body/>
-  </link>
+  <!-- No cam_1_link: cam_1 IS <camera_name>_camera_link from the ZED macro above.
+       A separate placeholder would be a second frame for one physical camera, which
+       is exactly the duplication this file used to have.
+       cam_2 is still a placeholder box: it is the planned second camera and nothing
+       publishes into it yet. When a real second ZED is added, instantiate the macro
+       again with a different `name` and delete this link. -->
   <link name="cam_2_link">
     <xacro:zedx_body/>
@@ -178,10 +218,7 @@
     <origin xyz="0 0 0.33" rpy="0 0 0"/>
   </joint>
-  <joint name="cam_1_joint" type="fixed">
-    <parent link="base_link"/>
-    <child link="cam_1_link"/>
-    <!-- Stern side (same side as props/rudder): boresight faces +Y (aft). -->
-    <origin xyz="${cam_x} ${cam_y} ${cam_z}" rpy="0 0 0"/>
-  </joint>
+  <!-- cam_1's mount is expressed once, inverted, as cam_1_to_base_link near the top
+       of this file (the camera is the root). There is deliberately no cam_1_joint
+       here: two joints for one mount is how the offset drifts. -->
   <joint name="cam_2_joint" type="fixed">
     <parent link="base_link"/>
