Commit message: feat: enhance URDF for Loon-E ASV with detailed links, joints, and geometry

File: loone_asv.export.urdf (robot description, URDF)
Before this commit: robot loone_asv, 5 links, 4 joints
Links:
- link base_link: geometry collision box size=1.0 0.6 0.2; visual box size=1.0 0.6 0.2
Joints:
- joint prop_l_joint: axis 1 0 0 -> 0 0 1; origin xyz=${prop_x} ${prop_y} 0 rpy=1.5708 0 0 -> xyz=-0.45 0.25 0 rpy=0 0 1.5708
- joint prop_r_joint: axis 1 0 0 -> 0 0 1; origin xyz=${prop_x} ${-prop_y} 0 rpy=1.5708 0 0 -> xyz=-0.45 -0.25 0 rpy=0 0 1.5708
- joint rudder_joint: origin xyz=${rudder_x} 0 0 rpy=0 0 1.5708 -> xyz=-0.55 0 0 rpy=0 0 1.5708

File: urdf/le1000_urdf_t4.urdf.xacro (robot description, xacro)
@@ -145,8 +145,9 @@
       <origin
         xyz="0 0 0"
-        rpy="0 0 0" />
-      <geometry>
-        <mesh
-          filename="package://le1000_urdf_t4/meshes/base_link.stl"/>
+        rpy="0 0 1.5708"/>
+      <geometry>
+        <mesh
+          filename="package://le1000_urdf_t4/meshes/base_link.stl"
+          />
       </geometry>
       <material
